Commit message: fix&perf: 修复遥控/仿真/模型/编译脚本bug，优化导航避障浮点运算与传参性能

File: src/diff_robot_description/urdf/diff_robot.urdf.xacro (robot description, xacro)
@@ -95,8 +95,10 @@
     </inertial>
   </link>
-  <joint name="caster_joint" type="fixed">
+  <joint name="caster_joint" type="continuous">
     <parent link="base_link"/>
     <child link="caster_wheel"/>
     <origin xyz="${-chassis_length/2 + 0.05} 0 ${-chassis_height/2}" rpy="0 0 0"/>
+    <axis xyz="1 0 0"/>
+    <dynamics damping="0.5" friction="0.1"/>
   </joint>
 </robot>

Commit message: fix: 补充URDF ros2_control标签与Gazebo控制插件，解决控制器启动失败、底盘无响应问题

File: src/diff_robot_description/urdf/diff_robot.urdf.xacro (robot description, xacro)
@@ -75,4 +75,32 @@
   <xacro:wheel prefix="left" y_offset="${wheel_separation/2}"/>
   <xacro:wheel prefix="right" y_offset="${-wheel_separation/2}"/>
+  <!-- ros2_control 硬件接口 -->
+  <ros2_control name="GazeboSystem" type="system">
+    <hardware>
+      <plugin>gazebo_ros2_control/GazeboSystem</plugin>
+    </hardware>
+    <joint name="left_wheel_joint">
+      <command_interface name="velocity">
+        <min>-1.0</min>
+        <max>1.0</max>
+      </command_interface>
+      <state_interface name="position"/>
+      <state_interface name="velocity"/>
+    </joint>
+    <joint name="right_wheel_joint">
+      <command_interface name="velocity">
+        <min>-1.0</min>
+        <max>1.0</max>
+      </command_interface>
+      <state_interface name="position"/>
+      <state_interface name="velocity"/>
+    </joint>
+  </ros2_control>
+  <!-- Gazebo ros2_control 插件 -->
+  <gazebo>
+    <plugin name="gazebo_ros2_control" filename="libgazebo_ros2_control.so">
+      <parameters>$(find diff_robot_control)/config/diff_robot_controllers.yaml</parameters>
+    </plugin>
+  </gazebo>
   <!-- 万向轮 -->
   <link name="caster_wheel">
